File: micro17.kicad_sch (KiCad schematic)
At the start: 55 parts, among them U1 AMS1117-3.3, U2 AMS1117-5.0, U3 STM32F405RGTx, U4 MCP6002, U5 MCP6002, Y1 8 MHz

Commit message: cleanup
Parts:
- removed C1, C25, C7: 22u/25V, Capacitor_SMD:C_0805_2012Metric, symbol Device:C
- removed C10, C11, C12, C15, C16, C17, C24, C5, C8: 100n, Capacitor_SMD:C_0603_1608Metric, symbol Device:C
- removed C13: 4n7, Capacitor_SMD:C_0603_1608Metric, symbol Device:C
- removed C14, C21: 10n, Capacitor_SMD:C_0603_1608Metric, symbol Device:C
- removed C18: 220p, Capacitor_SMD:C_0603_1608Metric, symbol Device:C
- removed C19: 680p, Capacitor_SMD:C_0603_1608Metric, symbol Device:C
- removed C2, C3: 2p2, Capacitor_SMD:C_0603_1608Metric, symbol Device:C
- removed C20: 1n5, Capacitor_SMD:C_0603_1608Metric, symbol Device:C
- removed C22, C23: 1u, Capacitor_SMD:C_0603_1608Metric, symbol Device:C
- removed C4, C6, C9: 2u2, Capacitor_SMD:C_0603_1608Metric, symbol Device:C
- removed D1, D2: DNP, symbol Device:LED
- removed J1, J2, J3, J4: ~, TestPoint:TestPoint_Pad_D1.5mm, symbol Connector_Generic:Conn_01x01
- removed R1, R13: 36k, Resistor_SMD:R_0603_1608Metric, symbol Device:R_Small
- removed R10: 130k, Resistor_SMD:R_0603_1608Metric, symbol Device:R_Small
- removed R11: 39k, Resistor_SMD:R_0603_1608Metric, symbol Device:R_Small
- removed R12: 10R, Resistor_SMD:R_0603_1608Metric, symbol Device:R_Small
- removed R14: 3k9, Resistor_SMD:R_0603_1608Metric, symbol Device:R_Small
- removed R15, R3, R4, R5: 10k, Resistor_SMD:R_0603_1608Metric, symbol Device:R_Small
- removed R16: 2k2, Resistor_SMD:R_0603_1608Metric, symbol Device:R_Small
- removed R2: 12k, Resistor_SMD:R_0603_1608Metric, symbol Device:R_Small
- removed R6, R7: DNP, Resistor_SMD:R_0603_1608Metric, symbol Device:R_Small
- removed R8: 9k1, Resistor_SMD:R_0603_1608Metric, symbol Device:R_Small
- removed R9: 3k3, Resistor_SMD:R_0603_1608Metric, symbol Device:R_Small
- removed RV1: 50k, symbol Device:R_Potentiometer
- removed RV2: 50k, Potentiometer_SMD:Potentiometer_Bourns_3224J_Horizontal, symbol Device:R_Potentiometer
- removed U1: AMS1117-3.3, Package_TO_SOT_SMD:SOT-223-3_TabPin2, symbol Regulator_Linear:AMS1117-3.3
- removed U2: AMS1117-5.0, Package_TO_SOT_SMD:SOT-223-3_TabPin2, symbol Regulator_Linear:AMS1117-5.0
- removed U3: STM32F405RGTx, Package_QFP:LQFP-64_10x10mm_P0.5mm, symbol MCU_ST_STM32F4:STM32F405RGTx
- removed U4, U5: MCP6002, Package_DFN_QFN:DFN-8-1EP_3x2mm_P0.5mm_EP1.75x1.45mm, symbol Amplifier_Operational:MCP6002-xMC
- removed Y1: 8 MHz, Crystal:Crystal_SMD_3225-4Pin_3.2x2.5mm, symbol Device:Crystal_GND24_Small
Connections:
- no-connect marks 31 -> 0
Other:
- added sheet Filtering (fltrs.kicad_sch)
- added sheet MCU (mcu.kicad_sch)
- added sheet Pins (pins.kicad_sch)
- added sheet Power supply (psu.kicad_sch)
- note removed: "Note: castellated pads + THT"

Commit message: PA2 Bias add, USB conn add.
Other:
- title: Micro17 - OpenRTX on a Module -> Micro17 - OpenRTX on a Module for Icom Radios
Changed lines of the file:
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@@
 	(paper "A4")
 	(title_block
-		(title "Micro17 - OpenRTX on a Module")
-		(date "05.12.2023")
+		(title "Micro17 - OpenRTX on a Module for Icom Radios")
+		(date "04.03.2024")
 		(rev "A")
 		(company "Wojciech Kaczmarski SP5WWP et al.")
 		(comment 1 "M17 Project, OpenRTX")
+		(comment 2 "Mano ON6RF")
+		(comment 3 "Mutlu TA1MD")
 	)
 	(sheet

Commit message: cosmetic changes to the schematic layout
- R25 - DNP
- PDF render update
Other:
- company: Wojciech Kaczmarski SP5WWP et al. -> Wojciech SP5WWP, Mano ON6RF, Mutlu TA1MD et al.
- title: Micro17 - OpenRTX on a Module for Icom Radios -> Micro17 - OpenRTX on a Module for ICOM radios
Changed lines of the file:
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@@
 	(paper "A4")
 	(title_block
-		(title "Micro17 - OpenRTX on a Module for Icom Radios")
-		(date "04.03.2024")
+		(title "Micro17 - OpenRTX on a Module for ICOM radios")
+		(date "06.03.2024")
 		(rev "A")
-		(company "Wojciech Kaczmarski SP5WWP et al.")
+		(company "Wojciech SP5WWP, Mano ON6RF, Mutlu TA1MD et al.")
 		(comment 1 "M17 Project, OpenRTX")
-		(comment 2 "Mano ON6RF")
-		(comment 3 "Mutlu TA1MD")
 	)
 	(sheet
